File: control-surface-left/control-surface-left.brd (EAGLE design)
At the start: 128.3 x 61 mm, 92 parts, among them IC1 74HC595D, IC2 74HC595D, IC3 74HC595D, IC4 74HC595D

Commit message: mods
Parts:
- added C4: (no value), rcl:C0805
- moved C1 62.2 mm to (48.9, 9.53)
- moved C2 31.7 mm to (80.6, 9.53)
- moved C3 30.5 mm to (111.1, 9.53)
Connections:
- net GND: now also C4.2
- net VCC: now also C4.1
Routing:
- net N$73: track 35.9 -> 30.6 mm
- net GND: track 114.7 -> 117.6 mm, vias 10 -> 11
- net VCC: track 236.2 -> 238.9 mm
Other:
- board text added: "hotchk155"
- board text added: "meta-step control surface (L) rev 1"
- board text added: "six4pix.com/metastep"
