File: control-surface-right/control-surface-right.brd (EAGLE design)
At the start: 121.9 x 61 mm, 75 parts, among them IC1 74HC595D, IC2 74HC595D, IC3 74HC595D, IC4 74HC595D

Commit message: mods
Parts:
- moved C1 46.4 mm to (62.9, 11.4)
- moved C2 23.5 mm to (86.4, 11.4)
- moved C3 22.9 mm to (109.2, 11.4)
Routing:
- net N$27: track 162.5 -> 243.3 mm
- net N$15: track 0.00 -> 6.15 mm
- net CK: track 125.2 -> 127.5 mm
- net VCC: track 174.2 -> 175.5 mm
- net H: track 115.1 -> 114.1 mm
Other:
- board text added: "hotchk155"
- board text added: "meta-step control surfacr (R) rev 1"
- board text added: "six4pix.com/metastep"
