File: control-surface-right/control-surface-right.sch (EAGLE design)
At the start: 75 parts, among them IC1 74HC595D, IC2 74HC595D, IC3 74HC595D, IC4 74HC595D

Commit message: mods
Other:
- moved on the sheet: C1, C2, C3
Changed lines of the file:
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@@
 <part name="LD1" library="led" deviceset="LED" device="3MM"/>
 <part name="LD6" library="led" deviceset="LED" device="3MM"/>
-<part name="C1" library="rcl" deviceset="C-EU" device="C0805"/>
+<part name="C3" library="rcl" deviceset="C-EU" device="C0805"/>
 <part name="SUPPLY1" library="supply2" deviceset="GND" device=""/>
 <part name="P+1" library="supply1" deviceset="VCC" device=""/>
@@
 <part name="LD9" library="led" deviceset="LED" device="3MM"/>
 <part name="LD8" library="led" deviceset="LED" device="3MM"/>
-<part name="C2" library="rcl" deviceset="C-EU" device="C0805"/>
+<part name="C1" library="rcl" deviceset="C-EU" device="C0805"/>
 <part name="SUPPLY2" library="supply2" deviceset="GND" device=""/>
 <part name="P+2" library="supply1" deviceset="VCC" device=""/>
@@
 <part name="LD11" library="led" deviceset="LED" device="3MM"/>
 <part name="LD4" library="led" deviceset="LED" device="3MM"/>
-<part name="C3" library="rcl" deviceset="C-EU" device="C0805"/>
+<part name="C2" library="rcl" deviceset="C-EU" device="C0805"/>
 <part name="SUPPLY3" library="supply2" deviceset="GND" device=""/>
 <part name="P+3" library="supply1" deviceset="VCC" device=""/>
@@
 <instance part="LD6" gate="G$1" x="73.66" y="45.72" rot="R90"/>
 <instance part="IC1" gate="P" x="43.18" y="30.48" rot="R90"/>
-<instance part="C1" gate="G$1" x="43.18" y="27.94" rot="R90"/>
+<instance part="C3" gate="G$1" x="43.18" y="27.94" rot="R90"/>
 <instance part="SUPPLY1" gate="GND" x="58.42" y="25.4"/>
 <instance part="P+1" gate="VCC" x="22.86" y="35.56"/>
@@
 <instance part="LD8" gate="G$1" x="73.66" y="0" rot="R90"/>
 <instance part="IC2" gate="P" x="43.18" y="-15.24" rot="R90"/>
-<instance part="C2" gate="G$1" x="43.18" y="-17.78" rot="R90"/>
+<instance part="C1" gate="G$1" x="43.18" y="-17.78" rot="R90"/>
 <instance part="SUPPLY2" gate="GND" x="58.42" y="-20.32"/>
 <instance part="P+2" gate="VCC" x="22.86" y="-10.16"/>
@@
 <instance part="LD4" gate="G$1" x="73.66" y="-76.2" rot="R90"/>
 <instance part="IC3" gate="P" x="43.18" y="-91.44" rot="R90"/>
-<instance part="C3" gate="G$1" x="43.18" y="-93.98" rot="R90"/>
+<instance part="C2" gate="G$1" x="43.18" y="-93.98" rot="R90"/>
 <instance part="SUPPLY3" gate="GND" x="58.42" y="-96.52"/>
 <instance part="P+3" gate="VCC" x="22.86" y="-86.36"/>
@@
 <net name="VCC" class="0">
 <segment>
-<pinref part="C1" gate="G$1" pin="1"/>
+<pinref part="C3" gate="G$1" pin="1"/>
 <wire x1="40.64" y1="27.94" x2="27.94" y2="27.94" width="0.1524" layer="91"/>
 <wire x1="27.94" y1="27.94" x2="27.94" y2="30.48" width="0.1524" layer="91"/>
@@
 </segment>
 <segment>
-<pinref part="C2" gate="G$1" pin="1"/>
+<pinref part="C1" gate="G$1" pin="1"/>
 <wire x1="40.64" y1="-17.78" x2="27.94" y2="-17.78" width="0.1524" layer="91"/>
 <wire x1="27.94" y1="-17.78" x2="27.94" y2="-15.24" width="0.1524" layer="91"/>
@@
 </segment>
 <segment>
-<pinref part="C3" gate="G$1" pin="1"/>
+<pinref part="C2" gate="G$1" pin="1"/>
 <wire x1="40.64" y1="-93.98" x2="27.94" y2="-93.98" width="0.1524" layer="91"/>
 <wire x1="27.94" y1="-93.98" x2="27.94" y2="-91.44" width="0.1524" layer="91"/>
@@
 <net name="GND" class="0">
 <segment>
-<pinref part="C1" gate="G$1" pin="2"/>
+<pinref part="C3" gate="G$1" pin="2"/>
 <wire x1="48.26" y1="27.94" x2="53.34" y2="27.94" width="0.1524" layer="91"/>
 <wire x1="53.34" y1="27.94" x2="53.34" y2="30.48" width="0.1524" layer="91"/>
@@
 </segment>
 <segment>
-<pinref part="C2" gate="G$1" pin="2"/>
+<pinref part="C1" gate="G$1" pin="2"/>
 <wire x1="48.26" y1="-17.78" x2="53.34" y2="-17.78" width="0.1524" layer="91"/>
 <wire x1="53.34" y1="-17.78" x2="53.34" y2="-15.24" width="0.1524" layer="91"/>
@@
 </segment>
 <segment>
-<pinref part="C3" gate="G$1" pin="2"/>
+<pinref part="C2" gate="G$1" pin="2"/>
 <wire x1="48.26" y1="-93.98" x2="53.34" y2="-93.98" width="0.1524" layer="91"/>
 <wire x1="53.34" y1="-93.98" x2="53.34" y2="-91.44" width="0.1524" layer="91"/>
@@
 <wire x1="111.76" y1="50.8" x2="119.888" y2="50.8" width="0.1524" layer="91"/>
 <junction x="111.76" y="50.8"/>
+<label x="101.6" y="50.8" size="1.778" layer="95"/>
 </segment>
 <segment>
@@
 </segment>
 </net>
-<net name="N$92" class="0">
-<segment>
-<wire x1="147.32" y1="-63.5" x2="149.86" y2="-63.5" width="0.1524" layer="91"/>
-</segment>
-</net>
