File: main-board/main-board.brd (EAGLE design)
At the start: 91.4 x 52.7 mm, 91 parts, among them IC1 MEGA8-AI, IC2 LM324D, IC3 74AC14D, IC4 6N138, IC5 MCP4728_QUAD_DAC

Commit message: stuff
Parts:
- moved R2 6.66 mm to (28.8, 26.7)
- moved C4 6.10 mm to (41.3, 45.1), turned to 270 degrees
- moved R5 1.42 mm to (32.4, 31.8)
- moved R3 1.33 mm to (39.0, 31.8)
- moved R4 1.28 mm to (36.7, 31.8)
Connections:
- net GND: now also R2.1, R3.1, R4.1, R5.1; no longer IC2.10, IC2.12, IC2.3, IC2.5
- net N$13: now also IC2.10; no longer R2.1
- net N$15: now also IC2.5; no longer R4.1
- net N$18: now also IC2.12; no longer R5.1
- net N$19: now also IC2.3; no longer R3.1
Routing:
- net N$5: track 26.3 -> 45.5 mm, vias 0 -> 3
- net N$13: track 3.29 -> 18.0 mm
- net N$15: track 4.13 -> 17.5 mm
- net N$10: track 71.0 -> 59.7 mm, vias 3 -> 1
- net N$11: track 33.4 -> 44.0 mm, vias 1 -> 2
- net N$18: track 4.45 -> 14.9 mm
- net GND: track 112.4 -> 121.9 mm
- net N$19: track 6.09 -> 14.6 mm
- net N$8: track 39.5 -> 31.3 mm, vias 1 -> 2
- net N$6: track 51.3 -> 46.6 mm, vias 2 -> 1
- net N$7: track 42.7 -> 38.0 mm, vias 1 -> 2
- net 9V: track 72.7 -> 76.5 mm, vias 1 -> 2
- net N$12: track 28.6 -> 25.3 mm, vias 1 -> 0
- net N$16: track 29.4 -> 31.9 mm

Commit message: rotate pots
Parts:
- moved R5 26.1 mm to (12.7, 48.9), turned to 180 degrees
- moved R2 24.9 mm to (17.7, 48.9), turned to 180 degrees
- moved R4 22.3 mm to (22.5, 48.9), turned to 180 degrees
- moved R3 20.7 mm to (27.3, 48.9), turned to 180 degrees
- moved CV1 12.3 mm to (27.3, 37.8), turned to 90 degrees
- moved CV4 8.71 mm to (12.8, 37.8), turned to 90 degrees
- moved CV2 5.32 mm to (22.5, 37.8), turned to 90 degrees
- moved CV3 1.73 mm to (17.7, 37.8), turned to 90 degrees
Routing:
- net N$10: track 59.7 -> 17.1 mm
- net N$8: track 31.3 -> 56.1 mm, vias 2 -> 3
- net N$6: track 46.6 -> 29.2 mm
- net N$7: track 38.0 -> 23.4 mm, vias 2 -> 0
- net N$12: track 25.3 -> 32.1 mm, vias 0 -> 1
- net N$11: track 44.0 -> 49.0 mm, vias 2 -> 3
- net N$5: track 45.5 -> 43.0 mm, vias 3 -> 1
- net GND: track 121.9 -> 122.8 mm, vias 9 -> 10
- net N$16: track 31.9 -> 32.3 mm, vias 0 -> 1
