File: main-board/main-board.sch (EAGLE design)
At the start: 21 parts, among them IC1 MEGA8-AI, IC2 LMV324M

Commit message: in progress
Parts:
- added C10, C11, C12, C13, C14: (no value), rcl:CPOL-EUE2-5
- added C15, C16, C17, C18, C19, C20, C21, C22, C23, C24, C25, C6, C8, C9: (no value), rcl:C-EUC0805
- added CLKIN, CLKOUT, CV1IN, CV1OUT, CV2IN, CV2OUT, CV3OUT, DAT, GATEOUT1, GATEOUT2, GND1, GND2, GND3, GND4, GND5, GND6, K0, K1, K2, K3, K4, K5, KS0, KS0A, KS1, KS1A, KS2, KS2A, KS3, KS3A, KS4, KS4A, KS5, KS5A, KS6, KS6A, KS7, KS7A, LED0, LED1, LED2, LED_CLK, LED_CLK1, LED_DAT, LED_DAT1, LED_OE, LED_OE1, MIDI_IN4, MIDI_IN5, MIDI_OUT4, MIDI_OUT5, POTA, POTB, POTC, POTD, POTE, POTF, POTG, POTH, POTI, POTJ, VCC1, VCC2, VCC3: (no value), pinhead:PINHD-1X1
- added IC3, IC4: 4051D, 40xx:4051D
- added IC6: 74HC595D, 74xx-eu:74HC595D
- added IC8: 74AC14D, 74xx-eu:74AC14D
- added JP1: (no value), pinhead:PINHD-1X6
- added LED5: (no value), led:LED3MM
- added OK1: 6N138, optocoupler:6N138
- added R11, R12, R13, R14, R15, R16, R22, R23, R24, R25, R26, R27, R28, R29, R30, R31, R32, R33, R34: (no value), rcl:R-EU_R0805
- added R21: (no value), pot:TRIM_EU-RJ9W
- added S9: (no value), switch-omron:10-XX
- added U$12: LD1086, jason_eagle6:LD1086
- added U$13, U$14, U$15, U$16, U$17, U$4, U$5: 0805DIODE, jasons_stuff:0805DIODE
- added U$18: TAG_CONN_AVR, jasons_stuff:TAG_CONN_AVR
- added U1: (no value), microbuilder:LM1117SOT223-REFLOW
Connections:
- removed net +5V: C3.1, C4.1, C5.1, U$1.VDD, U$1.VREF, U$2.VDD, U$2.VREF, U$3.VDD, U$3.VREF
- removed net +9V: IC2P.V+
- new net 1: IC1.PB3(MOSI/OC2), LED2.1, U$18.MOSI
- new net 2: IC1.PB4(MISO), LED1.1, U$18.MISO
- new net 3: IC1.PB5(SCK), LED0.1, LED5.A, U$18.SCK
- new net 9V: C10.+, C13.+, C15.1, C18.1, U$12.IN, U1.IN
- new net CLKIN: IC1.PD2(INT0), IC8C.O
- new net CLKOUT: IC1.PD3(INT1), IC8A.I
- new net CV1: CV1OUT.1, R8.2
- new net DAT: DAT.1, IC1.PD4(XCK/T0), IC6A.SER
- new net GATE1OUT: IC1.PC2(ADC2), IC8B.I
- new net GATE2OUT: IC1.PC3(ADC3), IC8D.I
- new net KS_CLK: IC1.PD5(T1), IC6A.RCK, IC6A.SCK
- new net LED_CLK: IC1.PD6(AIN0), LED_CLK.1, LED_CLK1.1
- new net LED_OE: IC1.PD7(AIN1), LED_OE.1, LED_OE1.1
- new net MIDI_IN: IC1.PD0(RXD), JP1.3, OK1.VO, R25.1
- new net MIDI_OUT: IC1.PD1(TXD), JP1.2, R27.2
- new net N$16: IC3A.X5, K0.1, R16.2
- new net N$18: IC3A.X4, POTE.1
- new net N$19: IC3A.X3, POTD.1
- new net N$20: IC3A.X2, POTC.1
- new net N$21: IC3A.X1, POTB.1
- new net N$22: IC3A.X0, POTA.1
- new net N$23: IC4A.X7, K5.1
- new net N$24: IC4A.X6, K4.1, R11.2
- new net N$26: IC6A.QC, KS2.1, KS2A.1
- new net N$27: IC6A.QD, KS3.1, KS3A.1
- new net N$28: IC6A.QE, KS4.1, KS4A.1
- new net N$29: IC6A.QF, KS5.1, KS5A.1
- new net N$30: IC6A.QG, KS6.1, KS6A.1
- new net N$31: IC6A.QH, KS7.1, KS7A.1
- new net N$32: IC4A.X5, K3.1, R12.2
- new net N$33: IC4A.X4, POTJ.1, R13.2
- new net N$34: IC4A.X3, POTI.1
- new net N$35: IC4A.X2, POTH.1
- new net N$36: IC4A.X1, POTG.1
- new net N$37: IC4A.X0, POTF.1
- new net N$38: LED_DAT.1, LED_DAT1.1
- new net N$39: MIDI_IN5.1, OK1.C, U$13.P$1
- new net N$50: IC6A.QA, KS0.1, KS0A.1
- new net N$54: OK1.A, R23.2, U$13.P$2
- new net N$55: C11.+, R21.E, R21.S, R22.2, U1.ADJ
- new net N$56: MIDI_IN4.1, R23.1
- new net N$57: OK1.VB, R24.1
- new net N$58: MIDI_OUT4.1, R26.1
- new net N$59: MIDI_OUT5.1, R27.1
- new net N$60: C22.1, IC8C.I, R30.1, U$4.P$1, U$5.P$2
- new net N$61: IC8B.O, R29.1
- new net N$62: IC8A.O, R28.1
- new net N$63: C19.1, CLKOUT.1, R28.2
- new net N$64: C20.1, GATEOUT1.1, R29.2
- new net N$65: CLKIN.1, R30.2
- new net N$66: IC8D.O, R31.1
- new net N$67: C21.1, GATEOUT2.1, R31.2
- new net N$68: CV1IN.1, R32.1
- new net N$69: CV2IN.1, R33.1
- new net N$71: LED5.C, R34.2
- new net N$72: CV3OUT.1, R10.2
- new net N$73: CV2OUT.1, R9.2
- new net N$8: IC3A.X7, K2.1, R14.2
- new net N$9: IC3A.X6, K1.1, R15.2
- new net PRG_RST: C23.2, JP1.1
- new net READ0: IC1.PC0(ADC0), IC3A.X
- new net READ1: IC1.PC1(ADC1), IC4A.X
- new net RESET: C23.1, IC1.PC6(/RESET), R1.2, S9.S, S9.S1, U$18.RESET
- new net SELA: IC1.PB0(ICP), IC3A.A, IC4A.A
- new net SELB: IC1.PB1(OC1A), IC3A.B, IC4A.B
- new net SELC: IC1.PB2(SS/OC1B), IC3A.C, IC4A.C
- new net VCC: C14.+, C16.1, C3.1, C4.1, C5.1, C6.1, C8.1, C9.1, IC1.AREF, IC1.AVCC, IC1.VCC@1, IC1.VCC@2, IC3P.VCC, IC4P.VCC, IC6A.SCL, IC6P.VCC, IC8P.VCC, OK1.VCC, R1.1, R25.2, R26.2, U$1.VDD, U$1.VREF, U$12.OUT, U$14.P$2, U$15.P$2, U$18.VCC, U$2.VDD, U$2.VREF, U$3.VDD, U$3.VREF, U$4.P$2, VCC1.1, VCC2.1, VCC3.1
- new net VREF: C12.+, C17.1, IC2P.V+, R22.1, U1.OUT
- net GND: now also C1.1, C10.-, C11.-, C12.-, C13.-, C14.-, C15.2, C16.2, C17.2, C18.2, C19.2, C2.1, C20.2, C21.2, C22.2, C24.1, C25.1, C6.2, C8.2, C9.2, GND1.1, GND2.1, GND3.1, GND4.1, GND5.1, GND6.1, IC1.GND, IC1.GND@1, IC1.GND@2, IC3A.INH, IC3P.GND, IC3P.VEE, IC4A.INH, IC4P.GND, IC4P.VEE, IC6A.G, IC6P.GND, IC8P.GND, JP1.5, JP1.6, OK1.GND, R11.1, R12.1, R13.1, R14.1, R15.1, R16.1, R21.A, R24.2, R34.1, S9.P, S9.P1, U$12.GND, U$16.P$1, U$17.P$1, U$18.GND, U$5.P$1
- net N$3: now also C24.2, IC1.ADC6, R32.2, U$14.P$1, U$16.P$2, U$17.P$2; no longer C1.1, C2.1, IC1.GND, IC1.GND@1, IC1.GND@2
- net N$4: now also C25.2, IC1.ADC7, R33.2, U$15.P$1; no longer IC1.AREF, IC1.AVCC, IC1.VCC@1, IC1.VCC@2, R1.1
- net N$5: now also IC6A.QB, KS1.1, KS1A.1; no longer IC1.PC6(/RESET), R1.2
- net SCL: now also IC1.PC5(ADC5/SCL)
- net SDA: now also IC1.PC4(ADC4/SDA)

Commit message: mode mods
Parts:
- removed C10, C11, C12: (no value), rcl:CPOL-EUE2-5
- removed C17, C18, C6, C8, C9: (no value), rcl:C-EUC0805
- removed GND2, GND5, GND6, K0, K1, K2, K3, K4, K5, KS0, KS0A, KS1, KS1A, KS2, KS2A, KS3, KS3A, KS4, KS4A, KS5, KS5A, KS6, KS6A, KS7, KS7A, LED_CLK, LED_CLK1, LED_DAT, LED_DAT1, LED_OE, LED_OE1, POTA, POTB, POTC, POTD, POTE, POTF, POTG, POTH, POTI, POTJ, VCC1, VCC2, VCC3: (no value), pinhead:PINHD-1X1
- removed IC3, IC4: 4051D, 40xx:4051D
- removed IC6: 74HC595D, 74xx-eu:74HC595D
- removed R12, R13, R14, R15, R16, R22, R7: (no value), rcl:R-EU_R0805
- removed R21: (no value), pot:TRIM_EU-RJ9W
- removed U1: (no value), microbuilder:LM1117SOT223-REFLOW
- added 9V, A, B, C, GND, GND0, KCK, LCK, LOE, RD0, RD1, VCC: (no value), pinhead:PINHD-1X1
- IC2: value LMV324M -> LM324D; device linear:LMV324M -> linear:LM324D
- R11, R5, R6: device rcl:R-EU_R0805 -> pot:TRIM_EU-RJ9W
- renumbered LED0 to L0, LED1 to L1, LED2 to L2
Connections:
- removed net N$16: IC3A.X5, K0.1, R16.2
- removed net N$18: IC3A.X4, POTE.1
- removed net N$19: IC3A.X3, POTD.1
- removed net N$20: IC3A.X2, POTC.1
- removed net N$21: IC3A.X1, POTB.1
- removed net N$22: IC3A.X0, POTA.1
- removed net N$23: IC4A.X7, K5.1
- removed net N$24: IC4A.X6, K4.1, R11.2
- removed net N$26: IC6A.QC, KS2.1, KS2A.1
- removed net N$27: IC6A.QD, KS3.1, KS3A.1
- removed net N$28: IC6A.QE, KS4.1, KS4A.1
- removed net N$29: IC6A.QF, KS5.1, KS5A.1
- removed net N$30: IC6A.QG, KS6.1, KS6A.1
- removed net N$31: IC6A.QH, KS7.1, KS7A.1
- removed net N$32: IC4A.X5, K3.1, R12.2
- removed net N$33: IC4A.X4, POTJ.1, R13.2
- removed net N$34: IC4A.X3, POTI.1
- removed net N$35: IC4A.X2, POTH.1
- removed net N$36: IC4A.X1, POTG.1
- removed net N$37: IC4A.X0, POTF.1
- removed net N$38: LED_DAT.1, LED_DAT1.1
- removed net N$5: IC6A.QB, KS1.1, KS1A.1
- removed net N$50: IC6A.QA, KS0.1, KS0A.1
- removed net N$55: C11.+, R21.E, R21.S, R22.2, U1.ADJ
- removed net N$8: IC3A.X7, K2.1, R14.2
- removed net N$9: IC3A.X6, K1.1, R15.2
- removed net READ0: IC1.PC0(ADC0), IC3A.X
- removed net READ1: IC1.PC1(ADC1), IC4A.X
- removed net VREF: C12.+, C17.1, IC2P.V+, R22.1, U1.OUT
- new net RD0: IC1.PC0(ADC0), RD0.1
- new net RD1: IC1.PC1(ADC1), RD1.1
- net 9V: now also 9V.1, IC2P.V+; no longer C10.+, C18.1, U1.IN
- net DAT: no longer IC6A.SER
- net GND: now also GND.1, GND0.1; no longer C10.-, C11.-, C12.-, C17.2, C18.2, C6.2, C8.2, C9.2, GND2.1, GND5.1, GND6.1, IC3A.INH, IC3P.GND, IC3P.VEE, IC4A.INH, IC4P.GND, IC4P.VEE, IC6A.G, IC6P.GND, R11.1, R12.1, R13.1, R14.1, R15.1, R16.1, R21.A
- net KS_CLK: now also KCK.1; no longer IC6A.RCK, IC6A.SCK
- net LED_CLK: now also LCK.1; no longer LED_CLK.1, LED_CLK1.1
- net LED_OE: now also LOE.1; no longer LED_OE.1, LED_OE1.1
- net N$10: now also R5.A; no longer R6.1
- net N$11: now also R6.E, R6.S; no longer R7.2
- net N$12: now also R5.E, R5.S; no longer R6.2
- net N$17: now also R11.E, R11.S; no longer R5.2
- net N$3: no longer U$17.P$2
- net N$4: now also U$17.P$2
- net N$6: now also R11.A; no longer R5.1
- net N$7: now also R6.A; no longer R7.1
- net SELA: now also A.1; no longer IC3A.A, IC4A.A
- net SELB: now also B.1; no longer IC3A.B, IC4A.B
- net SELC: now also C.1; no longer IC3A.C, IC4A.C
- net VCC: now also VCC.1; no longer C6.1, C8.1, C9.1, IC3P.VCC, IC4P.VCC, IC6A.SCL, IC6P.VCC, VCC1.1, VCC2.1, VCC3.1
Other:
- moved on the sheet: GND1, GND3, GND4

Commit message: stuff
Parts:
- renumbered GND0 to GD, IC8 to IC3, JP1 to SERIAL, LED5 to DIAG, OK1 to IC4, R11 to ADJ2, R5 to ADJ1, R6 to ADJ3, S9 to RESET, U$1 to DAC2, U$12 to REG1, U$13 to D1, U$14 to D3, U$15 to D5, U$16 to D2, U$17 to D4, U$18 to ICSP, U$2 to DAC1, U$3 to DAC0, U$4 to D7, U$5 to D6
Connections:
- net CV1: now also CV2OUT.1; no longer CV1OUT.1
- net GND: now also IC2D.+IN, IC2D.-IN
- net N$73: now also CV1OUT.1; no longer CV2OUT.1
- net VCC: now also IC3E.I, IC3F.I
Other:
- moved on the sheet: CV1OUT, CV2OUT

Commit message: stuff
Parts:
- removed ADJ1, ADJ2, ADJ3: (no value), pot:TRIM_EU-RJ9W
- removed C5: (no value), rcl:C-EUC0805
- removed DAC0, DAC1, DAC2: MCP4726, jasons_stuff:MCP4726
- added CV1, CV2, CV3, CV4: (no value), resistor:R-TRIMM3006P
- added CVO4: (no value), pinhead:PINHD-1X1
- added IC5: MCP4728_QUAD_DAC, jason_eagle6:MCP4728_QUAD_DAC
- added R5, R6: (no value), rcl:R-EU_R0805
- renumbered CLKIN to CKI, CLKOUT to CKO, CV1IN to CVI1, CV1OUT to CVO1, CV2IN to CVI2, CV2OUT to CVO2, CV3OUT to CVO3, GATEOUT1 to GT1, GATEOUT2 to GT2, MIDI_IN4 to MDI4, MIDI_IN5 to MDI5, MIDI_OUT4 to MDO4, MIDI_OUT5 to MDO5
Connections:
- removed net N$14: DAC1.VOUT, R3.1
- removed net N$17: ADJ2.E, ADJ2.S, IC2A.OUT, R8.1
- new net N$16: CV4.E, IC2D.-IN, R5.2
- new net N$18: IC5.VOUTD, R5.1
- new net N$19: IC5.VOUTA, R3.1
- new net N$5: CV3.A, CV3.S, IC2C.OUT, R10.1
- new net N$8: CV4.A, CV4.S, IC2D.OUT, R6.1
- new net N$9: CVO4.1, R6.2
- net 9V: now also C4.2
- net GND: now also C3.1, C4.1, IC5.LDAC#, IC5.VSS; no longer C3.2, C4.2, C5.2, DAC0.VSS, DAC1.VSS, DAC2.VSS, IC2D.-IN
- net N$10: now also CV1.E; no longer ADJ1.A
- net N$11: now also CV2.A, CV2.S, IC2A.OUT, R8.1; no longer ADJ3.E, ADJ3.S, IC2C.OUT, R10.1
- net N$12: now also CV1.A, CV1.S; no longer ADJ1.E, ADJ1.S
- net N$13: now also IC5.VOUTC; no longer DAC0.VOUT
- net N$15: now also IC5.VOUTB; no longer DAC2.VOUT
- net N$6: now also CV2.E; no longer ADJ2.A
- net N$7: now also CV3.E; no longer ADJ3.A
- net SCL: now also IC5.SCL; no longer DAC0.SCL, DAC1.SCL, DAC2.SCL
- net SDA: now also IC5.SDA; no longer DAC0.SDA, DAC1.SDA, DAC2.SDA
- net VCC: now also C3.2, IC5.VDD; no longer C3.1, C4.1, C5.1, DAC0.VDD, DAC0.VREF, DAC1.VDD, DAC1.VREF, DAC2.VDD, DAC2.VREF
Other:
- moved on the sheet: C3, C4, IC2D

Commit message: stuff
Connections:
- net GND: now also R2.1, R3.1, R4.1, R5.1; no longer IC2A.+IN, IC2B.+IN, IC2C.+IN, IC2D.+IN
- net N$13: now also IC2C.+IN; no longer R2.1
- net N$15: now also IC2B.+IN; no longer R4.1
- net N$18: now also IC2D.+IN; no longer R5.1
- net N$19: now also IC2A.+IN; no longer R3.1
Changed lines of the file:
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@@
 <wire x1="441.96" y1="144.78" x2="414.02" y2="144.78" width="0.1524" layer="91"/>
 <junction x="414.02" y="144.78"/>
-<pinref part="IC2" gate="A" pin="+IN"/>
-<wire x1="434.34" y1="160.02" x2="414.02" y2="160.02" width="0.1524" layer="91"/>
-<wire x1="414.02" y1="160.02" x2="414.02" y2="144.78" width="0.1524" layer="91"/>
-<wire x1="414.02" y1="139.7" x2="414.02" y2="144.78" width="0.1524" layer="91"/>
-<pinref part="IC2" gate="B" pin="+IN"/>
-<wire x1="434.34" y1="139.7" x2="414.02" y2="139.7" width="0.1524" layer="91"/>
-<junction x="414.02" y="139.7"/>
-<pinref part="IC2" gate="C" pin="+IN"/>
-<wire x1="434.34" y1="121.92" x2="414.02" y2="121.92" width="0.1524" layer="91"/>
-<wire x1="414.02" y1="121.92" x2="414.02" y2="139.7" width="0.1524" layer="91"/>
-<pinref part="IC2" gate="D" pin="+IN"/>
-<wire x1="434.34" y1="93.98" x2="414.02" y2="93.98" width="0.1524" layer="91"/>
-<wire x1="414.02" y1="93.98" x2="414.02" y2="121.92" width="0.1524" layer="91"/>
-<junction x="414.02" y="121.92"/>
-<wire x1="414.02" y1="160.02" x2="414.02" y2="175.26" width="0.1524" layer="91"/>
-<junction x="414.02" y="160.02"/>
-<junction x="434.34" y="160.02"/>
-<junction x="434.34" y="139.7"/>
-<junction x="434.34" y="121.92"/>
-<junction x="434.34" y="93.98"/>
+<wire x1="414.02" y1="88.9" x2="414.02" y2="116.84" width="0.1524" layer="91"/>
+<wire x1="414.02" y1="116.84" x2="414.02" y2="134.62" width="0.1524" layer="91"/>
+<wire x1="414.02" y1="134.62" x2="414.02" y2="144.78" width="0.1524" layer="91"/>
+<wire x1="414.02" y1="144.78" x2="414.02" y2="154.94" width="0.1524" layer="91"/>
 <label x="414.02" y="175.26" size="1.778" layer="95"/>
+<pinref part="R5" gate="G$1" pin="1"/>
+<wire x1="414.02" y1="154.94" x2="414.02" y2="175.26" width="0.1524" layer="91"/>
+<wire x1="419.1" y1="88.9" x2="414.02" y2="88.9" width="0.1524" layer="91"/>
+<pinref part="R2" gate="G$1" pin="1"/>
+<wire x1="419.1" y1="116.84" x2="414.02" y2="116.84" width="0.1524" layer="91"/>
+<junction x="414.02" y="116.84"/>
+<pinref part="R3" gate="G$1" pin="1"/>
+<wire x1="419.1" y1="134.62" x2="414.02" y2="134.62" width="0.1524" layer="91"/>
+<junction x="414.02" y="134.62"/>
+<pinref part="R4" gate="G$1" pin="1"/>
+<wire x1="419.1" y1="154.94" x2="414.02" y2="154.94" width="0.1524" layer="91"/>
+<junction x="414.02" y="154.94"/>
 </segment>
 <segment>
@@
 <segment>
 <pinref part="R4" gate="G$1" pin="2"/>
-<pinref part="IC2" gate="A" pin="-IN"/>
 <wire x1="429.26" y1="154.94" x2="431.8" y2="154.94" width="0.1524" layer="91"/>
-<wire x1="431.8" y1="154.94" x2="434.34" y2="154.94" width="0.1524" layer="91"/>
 <wire x1="431.8" y1="147.32" x2="431.8" y2="154.94" width="0.1524" layer="91"/>
-<junction x="431.8" y="154.94"/>
 <junction x="429.26" y="154.94"/>
 <pinref part="CV2" gate="G$1" pin="E"/>
 <wire x1="447.04" y1="147.32" x2="431.8" y2="147.32" width="0.1524" layer="91"/>
+<pinref part="IC2" gate="A" pin="-IN"/>
+<wire x1="431.8" y1="154.94" x2="434.34" y2="154.94" width="0.1524" layer="91"/>
+<junction x="431.8" y="154.94"/>
 </segment>
 </net>
@@
 </segment>
 </net>
-<net name="N$13" class="0">
-<segment>
-<pinref part="R2" gate="G$1" pin="1"/>
-<pinref part="IC5" gate="G$1" pin="VOUTC"/>
-<wire x1="383.54" y1="116.84" x2="419.1" y2="116.84" width="0.1524" layer="91"/>
-<junction x="383.54" y="116.84"/>
-<junction x="419.1" y="116.84"/>
-</segment>
-</net>
 <net name="N$15" class="0">
 <segment>
-<pinref part="R4" gate="G$1" pin="1"/>
 <pinref part="IC5" gate="G$1" pin="VOUTB"/>
 <wire x1="383.54" y1="114.3" x2="396.24" y2="114.3" width="0.1524" layer="91"/>
-<wire x1="396.24" y1="114.3" x2="396.24" y2="154.94" width="0.1524" layer="91"/>
-<wire x1="396.24" y1="154.94" x2="419.1" y2="154.94" width="0.1524" layer="91"/>
 <junction x="383.54" y="114.3"/>
-<junction x="419.1" y="154.94"/>
+<wire x1="396.24" y1="114.3" x2="396.24" y2="139.7" width="0.1524" layer="91"/>
+<pinref part="IC2" gate="B" pin="+IN"/>
+<wire x1="396.24" y1="139.7" x2="434.34" y2="139.7" width="0.1524" layer="91"/>
 </segment>
 </net>
@@
 <net name="N$18" class="0">
 <segment>
-<pinref part="R5" gate="G$1" pin="1"/>
-<wire x1="419.1" y1="88.9" x2="401.32" y2="88.9" width="0.1524" layer="91"/>
 <pinref part="IC5" gate="G$1" pin="VOUTD"/>
 <wire x1="383.54" y1="119.38" x2="401.32" y2="119.38" width="0.1524" layer="91"/>
-<wire x1="401.32" y1="119.38" x2="401.32" y2="88.9" width="0.1524" layer="91"/>
+<wire x1="401.32" y1="119.38" x2="401.32" y2="93.98" width="0.1524" layer="91"/>
 <junction x="383.54" y="119.38"/>
-<junction x="419.1" y="88.9"/>
+<pinref part="IC2" gate="D" pin="+IN"/>
+<wire x1="434.34" y1="93.98" x2="401.32" y2="93.98" width="0.1524" layer="91"/>
 </segment>
 </net>
@@
 <pinref part="IC5" gate="G$1" pin="VOUTA"/>
 <wire x1="383.54" y1="111.76" x2="398.78" y2="111.76" width="0.1524" layer="91"/>
-<wire x1="398.78" y1="111.76" x2="398.78" y2="134.62" width="0.1524" layer="91"/>
+<wire x1="398.78" y1="111.76" x2="398.78" y2="160.02" width="0.1524" layer="91"/>
 <junction x="383.54" y="111.76"/>
-<pinref part="R3" gate="G$1" pin="1"/>
-<wire x1="398.78" y1="134.62" x2="419.1" y2="134.62" width="0.1524" layer="91"/>
+<pinref part="IC2" gate="A" pin="+IN"/>
+<wire x1="434.34" y1="160.02" x2="398.78" y2="160.02" width="0.1524" layer="91"/>
 </segment>
 </net>
@@
 </segment>
 </net>
+<net name="N$13" class="0">
+<segment>
+<pinref part="IC5" gate="G$1" pin="VOUTC"/>
+<wire x1="383.54" y1="116.84" x2="408.94" y2="116.84" width="0.1524" layer="91"/>
+<wire x1="408.94" y1="116.84" x2="408.94" y2="121.92" width="0.1524" layer="91"/>
+<pinref part="IC2" gate="C" pin="+IN"/>
+<wire x1="408.94" y1="121.92" x2="434.34" y2="121.92" width="0.1524" layer="91"/>
+</segment>
+</net>
