File: pots-board/pots-board.sch (EAGLE design)
At the start: 29 parts

Commit message: mods
Parts:
- renumbered A to POT1, B to POT2, C to POT3, D to POT4, E to POT5
Changed lines of the file:
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@@
 </classes>
 <parts>
-<part name="A" library="jasons_stuff" deviceset="ALPS_POT_SMALL" device=""/>
-<part name="B" library="jasons_stuff" deviceset="ALPS_POT_SMALL" device=""/>
-<part name="C" library="jasons_stuff" deviceset="ALPS_POT_SMALL" device=""/>
-<part name="D" library="jasons_stuff" deviceset="ALPS_POT_SMALL" device=""/>
-<part name="E" library="jasons_stuff" deviceset="ALPS_POT_SMALL" device=""/>
+<part name="POT1" library="jasons_stuff" deviceset="ALPS_POT_SMALL" device=""/>
+<part name="POT2" library="jasons_stuff" deviceset="ALPS_POT_SMALL" device=""/>
+<part name="POT3" library="jasons_stuff" deviceset="ALPS_POT_SMALL" device=""/>
+<part name="POT4" library="jasons_stuff" deviceset="ALPS_POT_SMALL" device=""/>
+<part name="POT5" library="jasons_stuff" deviceset="ALPS_POT_SMALL" device=""/>
 <part name="VC1" library="pinhead" deviceset="PINHD-1X1" device=""/>
 <part name="GD1" library="pinhead" deviceset="PINHD-1X1" device=""/>
@@
 </plain>
 <instances>
-<instance part="A" gate="G$1" x="25.4" y="40.64"/>
-<instance part="B" gate="G$1" x="48.26" y="40.64"/>
-<instance part="C" gate="G$1" x="68.58" y="40.64"/>
-<instance part="D" gate="G$1" x="88.9" y="40.64"/>
-<instance part="E" gate="G$1" x="109.22" y="40.64"/>
+<instance part="POT1" gate="G$1" x="25.4" y="40.64"/>
+<instance part="POT2" gate="G$1" x="48.26" y="40.64"/>
+<instance part="POT3" gate="G$1" x="68.58" y="40.64"/>
+<instance part="POT4" gate="G$1" x="88.9" y="40.64"/>
+<instance part="POT5" gate="G$1" x="109.22" y="40.64"/>
 <instance part="VC1" gate="G$1" x="2.54" y="58.42" rot="R180"/>
 <instance part="GD1" gate="G$1" x="2.54" y="27.94" rot="R180"/>
@@
 <segment>
 <pinref part="VC1" gate="G$1" pin="1"/>
-<pinref part="E" gate="G$1" pin="B"/>
+<pinref part="POT5" gate="G$1" pin="B"/>
 <wire x1="5.08" y1="58.42" x2="25.4" y2="58.42" width="0.1524" layer="91"/>
 <wire x1="25.4" y1="58.42" x2="48.26" y2="58.42" width="0.1524" layer="91"/>
@@
 <wire x1="88.9" y1="58.42" x2="109.22" y2="58.42" width="0.1524" layer="91"/>
 <wire x1="109.22" y1="58.42" x2="109.22" y2="53.34" width="0.1524" layer="91"/>
-<pinref part="D" gate="G$1" pin="B"/>
+<pinref part="POT4" gate="G$1" pin="B"/>
 <wire x1="88.9" y1="53.34" x2="88.9" y2="58.42" width="0.1524" layer="91"/>
 <junction x="88.9" y="58.42"/>
-<pinref part="C" gate="G$1" pin="B"/>
+<pinref part="POT3" gate="G$1" pin="B"/>
 <wire x1="68.58" y1="53.34" x2="68.58" y2="58.42" width="0.1524" layer="91"/>
 <junction x="68.58" y="58.42"/>
-<pinref part="B" gate="G$1" pin="B"/>
+<pinref part="POT2" gate="G$1" pin="B"/>
 <wire x1="48.26" y1="53.34" x2="48.26" y2="58.42" width="0.1524" layer="91"/>
 <junction x="48.26" y="58.42"/>
-<pinref part="A" gate="G$1" pin="B"/>
+<pinref part="POT1" gate="G$1" pin="B"/>
 <wire x1="25.4" y1="53.34" x2="25.4" y2="58.42" width="0.1524" layer="91"/>
 <junction x="25.4" y="58.42"/>
@@
 <segment>
 <pinref part="GD1" gate="G$1" pin="1"/>
-<pinref part="E" gate="G$1" pin="A"/>
+<pinref part="POT5" gate="G$1" pin="A"/>
 <wire x1="5.08" y1="27.94" x2="25.4" y2="27.94" width="0.1524" layer="91"/>
 <wire x1="25.4" y1="27.94" x2="48.26" y2="27.94" width="0.1524" layer="91"/>
@@
 <wire x1="88.9" y1="27.94" x2="109.22" y2="27.94" width="0.1524" layer="91"/>
 <wire x1="109.22" y1="27.94" x2="109.22" y2="33.02" width="0.1524" layer="91"/>
-<pinref part="D" gate="G$1" pin="A"/>
+<pinref part="POT4" gate="G$1" pin="A"/>
 <wire x1="88.9" y1="33.02" x2="88.9" y2="27.94" width="0.1524" layer="91"/>
 <junction x="88.9" y="27.94"/>
-<pinref part="C" gate="G$1" pin="A"/>
+<pinref part="POT3" gate="G$1" pin="A"/>
 <wire x1="68.58" y1="33.02" x2="68.58" y2="27.94" width="0.1524" layer="91"/>
 <junction x="68.58" y="27.94"/>
-<pinref part="B" gate="G$1" pin="A"/>
+<pinref part="POT2" gate="G$1" pin="A"/>
 <wire x1="48.26" y1="33.02" x2="48.26" y2="27.94" width="0.1524" layer="91"/>
 <junction x="48.26" y="27.94"/>
-<pinref part="A" gate="G$1" pin="A"/>
+<pinref part="POT1" gate="G$1" pin="A"/>
 <wire x1="25.4" y1="33.02" x2="25.4" y2="27.94" width="0.1524" layer="91"/>
 <junction x="25.4" y="27.94"/>
@@
 <net name="N$3" class="0">
 <segment>
-<pinref part="A" gate="G$1" pin="W"/>
+<pinref part="POT1" gate="G$1" pin="W"/>
 <wire x1="33.02" y1="43.18" x2="40.64" y2="43.18" width="0.1524" layer="91"/>
 <wire x1="40.64" y1="43.18" x2="40.64" y2="17.78" width="0.1524" layer="91"/>
@@
 <net name="N$4" class="0">
 <segment>
-<pinref part="B" gate="G$1" pin="W"/>
+<pinref part="POT2" gate="G$1" pin="W"/>
 <pinref part="VB" gate="G$1" pin="1"/>
 <wire x1="55.88" y1="43.18" x2="60.96" y2="43.18" width="0.1524" layer="91"/>
@@
 <net name="N$5" class="0">
 <segment>
-<pinref part="C" gate="G$1" pin="W"/>
+<pinref part="POT3" gate="G$1" pin="W"/>
 <pinref part="VC" gate="G$1" pin="1"/>
 <wire x1="76.2" y1="43.18" x2="81.28" y2="43.18" width="0.1524" layer="91"/>
@@
 <net name="N$6" class="0">
 <segment>
-<pinref part="D" gate="G$1" pin="W"/>
+<pinref part="POT4" gate="G$1" pin="W"/>
 <pinref part="VD" gate="G$1" pin="1"/>
 <wire x1="96.52" y1="43.18" x2="101.6" y2="43.18" width="0.1524" layer="91"/>
@@
 <net name="N$7" class="0">
 <segment>
-<pinref part="E" gate="G$1" pin="W"/>
+<pinref part="POT5" gate="G$1" pin="W"/>
 <pinref part="VE" gate="G$1" pin="1"/>
 <wire x1="116.84" y1="43.18" x2="124.46" y2="43.18" width="0.1524" layer="91"/>

Commit message: stuff
Parts:
- added C1, C2, C3, C4: (no value), rcl:C-EUC0805
Connections:
- removed net N$1: POT1.B, POT2.B, POT3.B, POT4.B, POT5.B, VC1.1, VCC.1, VCC10.1
- new net VCC: C1.1, C2.1, C3.1, C4.1, POT1.B, POT2.B, POT3.B, POT4.B, POT5.B, VC1.1, VCC.1, VCC10.1
- net GND: now also C1.2, C2.2, C3.2, C4.2
Changed lines of the file:
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@@
 <part name="GND50" library="pinhead" deviceset="PINHD-1X1" device=""/>
 <part name="VCC10" library="pinhead" deviceset="PINHD-1X1" device=""/>
+<part name="C1" library="rcl" deviceset="C-EU" device="C0805"/>
+<part name="C2" library="rcl" deviceset="C-EU" device="C0805"/>
+<part name="C3" library="rcl" deviceset="C-EU" device="C0805"/>
+<part name="C4" library="rcl" deviceset="C-EU" device="C0805"/>
 </parts>
 <sheets>
@@
 <instance part="GND50" gate="G$1" x="134.62" y="5.08"/>
 <instance part="VCC10" gate="G$1" x="134.62" y="50.8"/>
+<instance part="C1" gate="G$1" x="55.88" y="81.28"/>
+<instance part="C2" gate="G$1" x="63.5" y="81.28"/>
+<instance part="C3" gate="G$1" x="71.12" y="81.28"/>
+<instance part="C4" gate="G$1" x="78.74" y="81.28"/>
 </instances>
 <busses>
 </busses>
 <nets>
-<net name="N$1" class="0">
+<net name="VCC" class="0">
 <segment>
 <pinref part="VC1" gate="G$1" pin="1"/>
@@
 <wire x1="129.54" y1="50.8" x2="129.54" y2="58.42" width="0.1524" layer="91"/>
 <junction x="129.54" y="58.42"/>
+<label x="35.56" y="55.88" size="1.778" layer="95"/>
+</segment>
+<segment>
+<pinref part="C1" gate="G$1" pin="1"/>
+<wire x1="55.88" y1="83.82" x2="55.88" y2="91.44" width="0.1524" layer="91"/>
+<pinref part="C4" gate="G$1" pin="1"/>
+<wire x1="55.88" y1="91.44" x2="63.5" y2="91.44" width="0.1524" layer="91"/>
+<wire x1="63.5" y1="91.44" x2="71.12" y2="91.44" width="0.1524" layer="91"/>
+<wire x1="71.12" y1="91.44" x2="78.74" y2="91.44" width="0.1524" layer="91"/>
+<wire x1="78.74" y1="91.44" x2="78.74" y2="83.82" width="0.1524" layer="91"/>
+<pinref part="C3" gate="G$1" pin="1"/>
+<wire x1="71.12" y1="83.82" x2="71.12" y2="91.44" width="0.1524" layer="91"/>
+<junction x="71.12" y="91.44"/>
+<pinref part="C2" gate="G$1" pin="1"/>
+<wire x1="63.5" y1="83.82" x2="63.5" y2="91.44" width="0.1524" layer="91"/>
+<junction x="63.5" y="91.44"/>
+<wire x1="78.74" y1="91.44" x2="86.36" y2="91.44" width="0.1524" layer="91"/>
+<junction x="78.74" y="91.44"/>
+<label x="86.36" y="91.44" size="1.778" layer="95"/>
 </segment>
 </net>
@@
 <wire x1="132.08" y1="12.7" x2="129.54" y2="12.7" width="0.1524" layer="91"/>
 <junction x="129.54" y="12.7"/>
+<label x="33.02" y="27.94" size="1.778" layer="95"/>
+</segment>
+<segment>
+<pinref part="C1" gate="G$1" pin="2"/>
+<wire x1="55.88" y1="76.2" x2="55.88" y2="68.58" width="0.1524" layer="91"/>
+<pinref part="C4" gate="G$1" pin="2"/>
+<wire x1="55.88" y1="68.58" x2="63.5" y2="68.58" width="0.1524" layer="91"/>
+<wire x1="63.5" y1="68.58" x2="71.12" y2="68.58" width="0.1524" layer="91"/>
+<wire x1="71.12" y1="68.58" x2="78.74" y2="68.58" width="0.1524" layer="91"/>
+<wire x1="78.74" y1="68.58" x2="78.74" y2="76.2" width="0.1524" layer="91"/>
+<pinref part="C2" gate="G$1" pin="2"/>
+<wire x1="63.5" y1="76.2" x2="63.5" y2="68.58" width="0.1524" layer="91"/>
+<junction x="63.5" y="68.58"/>
+<pinref part="C3" gate="G$1" pin="2"/>
+<wire x1="71.12" y1="76.2" x2="71.12" y2="68.58" width="0.1524" layer="91"/>
+<junction x="71.12" y="68.58"/>
+<wire x1="78.74" y1="68.58" x2="86.36" y2="68.58" width="0.1524" layer="91"/>
+<junction x="78.74" y="68.58"/>
+<label x="86.36" y="68.58" size="1.778" layer="95"/>
 </segment>
 </net>
